Commit message: Urdf completo (gripers descargados)
El modelo del urdf ya tiene todas las articulaciones funcionando, falta ubicar las coberturas y  hay que ver si conviene poner limites a las articulaciones en el modelo

File: src/rhino_description/rhino_description/debug.urdf (robot description, URDF)
Before this commit: robot rhino, 19 links, 18 joints
Links:
- added link left_gripper; visual mesh filename=l_finger.dae
- added link mano; visual cylinder length=0.2 radius=0.01
- added link right_gripper; visual mesh filename=l_finger.dae
Joints:
- added joint gripper_izquierdo: type revolute, parent engranaje_muneca, child left_gripper, origin xyz=0 0.01 0 rpy=0 0 0, axis -1.0 0.0 0.0, limit lower=-0.38 upper=0 effort=1000.0 velocity=0.5
- added joint gripper_right: type revolute, parent engranaje_muneca, child right_gripper, origin xyz=0 -0.01 0 rpy=0 0 0, axis 10 0 0, limit lower=-0.38 upper=0 effort=1000.0 velocity=0.5
- added joint muneca_mano: type fixed, parent engranaje_muneca, child mano, origin xyz=0 0 -0.23
- joint codo_antebrazo: limit lower=1.7 upper=2.5 effort=1000.0 velocity=0.5 -> lower=-3.14 upper=3.14 effort=1000.0 velocity=0.5

Commit message: ....

File: src/rhino_description/rhino_description/debug.urdf (robot description, URDF)
Before this commit: robot rhino, 22 links, 21 joints
Links:
- removed link prueba
- removed link prueba1
- link cubierta_antebrazo1: geometry visual mesh filename=antebrazo.stl scale=0.001 0.001 0.001
- link cubierta_antebrazo2: geometry visual mesh filename=antebrazo.stl scale=0.001 0.001 0.001
- link cubierta_brazo1: geometry visual mesh filename=brazo.stl scale=0.001 0.001 0.001
- link cubierta_brazo2: geometry visual mesh filename=brazo.stl scale=0.001 0.001 0.001
- link left_gripper: geometry visual mesh filename=package://rhino_description/meshes/l_finger.dae
- link right_gripper: geometry visual mesh filename=package://rhino_description/meshes/l_finger.dae
Joints:
- removed joint tronco_to_prueba
- removed joint tronco_to_prueba1
