Commit message: Falta la mano

File: install/rhino_description/share/rhino_description/description/rhino.urdf (robot description, URDF)
Before this commit: robot rhino, 19 links, 18 joints
Links:
- removed link prueba
- removed link prueba1
- added link left_gripper; visual mesh filename=package://rhino_description/meshes/dedo.dae
- added link mano; visual cylinder length=0.2 radius=0.01
- added link right_gripper; visual mesh filename=package://rhino_description/meshes/dedo.dae
- link engranaje_muneca: geometry visual mesh filename=package://rhino_description/meshes/engranaje.stl scale=0.001 0.001 0.001
Joints:
- removed joint tronco_to_prueba
- removed joint tronco_to_prueba1
- added joint gripper_izquierdo: type revolute, parent engranaje_muneca, child left_gripper, origin xyz=0 0.01 0 rpy=0 0 0, axis -1.0 0.0 0.0, limit lower=-0.38 upper=0 effort=1000.0 velocity=0.5
- added joint gripper_right: type revolute, parent engranaje_muneca, child right_gripper, origin xyz=0 -0.01 0 rpy=0 0 0, axis 10 0 0, limit lower=-0.38 upper=0 effort=1000.0 velocity=0.5
- added joint muneca_mano: type fixed, parent engranaje_muneca, child mano, origin xyz=0 0 -0.23
- joint codo_antebrazo: limit lower=1.7 upper=2.5 effort=1000.0 velocity=0.5 -> lower=-3.14 upper=3.14 effort=1000.0 velocity=0.5

File: src/rhino_description/rhino_description/debug.urdf (robot description, URDF)
Before this commit: robot rhino, 20 links, 19 joints
Links:
- link engranaje_muneca: geometry visual mesh filename=Engranaje.stl scale=0.002 0.002 0.001
- link left_gripper: geometry visual mesh filename=l_finger.dae
- link muneca: geometry visual box size=0.1 0.07 0.2
- link right_gripper: geometry visual mesh filename=l_finger.dae

Commit message: Modelo con mano

File: install/rhino_description/share/rhino_description/description/rhino.urdf (robot description, URDF)
Before this commit: robot rhino, 20 links, 19 joints
Links:
- removed link mano
- link engranaje_muneca: geometry visual mesh filename=package://rhino_description/meshes/Engranaje.stl scale=0.001 0.001 0.001
- link left_gripper: geometry visual mesh filename=package://rhino_description/meshes/mano.stl scale=0.001 0.001 0.001
- link muneca: geometry visual box size=0.1 0.07 0.2
- link right_gripper: geometry visual mesh filename=package://rhino_description/meshes/mano.stl scale=0.001 0.001 0.001
Joints:
- removed joint muneca_mano
- joint gripper_izquierdo: limit lower=-0.38 upper=0 effort=1000.0 velocity=0.5 -> lower=-3.15 upper=0 effort=1000.0 velocity=0.5; origin xyz=0 0.01 0 rpy=0 0 0 -> xyz=0 0.01 -0.08 rpy=0 0 0
- joint gripper_right: limit lower=-0.38 upper=0 effort=1000.0 velocity=0.5 -> lower=-3.15 upper=0 effort=1000.0 velocity=0.5; origin xyz=0 -0.01 0 rpy=0 0 0 -> xyz=0 -0.01 -0.08 rpy=0 0 0

File: src/rhino_description/rhino_description/debug.urdf (robot description, URDF)
Before this commit: robot rhino, 20 links, 19 joints
Links:
- removed link mano
- link left_gripper: geometry visual mesh filename=mano.stl scale=0.001 0.001 0.001
- link right_gripper: geometry visual mesh filename=mano.stl scale=0.001 0.001 0.001
Joints:
- removed joint muneca_mano
- joint gripper_izquierdo: limit lower=-0.38 upper=0 effort=1000.0 velocity=0.5 -> lower=-3.15 upper=0 effort=1000.0 velocity=0.5; origin xyz=0 0.01 0 rpy=0 0 0 -> xyz=0 0.01 -0.08 rpy=0 0 0
- joint gripper_right: limit lower=-0.38 upper=0 effort=1000.0 velocity=0.5 -> lower=-3.15 upper=0 effort=1000.0 velocity=0.5; origin xyz=0 -0.01 0 rpy=0 0 0 -> xyz=0 -0.01 -0.08 rpy=0 0 0
